Commit message: added emily's compressed STL meshes, crab robot / noodle limbs loadsgit branch

File: robot_model/crab/rad_arm.urdf (robot description, URDF)
Before this commit: robot rad_arm, 15 links, 14 joints
Links:
- link cluster_1_distal_link: geometry collision mesh filename=package://meshes/776_meshes/distal_link.STL; visual mesh filename=package://meshes/776_meshes/distal_link.STL
- link cluster_1_end_link: geometry collision mesh filename=package://meshes/776_meshes/end_link.STL; visual mesh filename=package://meshes/776_meshes/end_link.STL
- link cluster_1_proximal_link: geometry collision mesh filename=package://meshes/776_meshes/proximal_link.STL; visual mesh filename=package://meshes/776_meshes/proximal_link.STL
- link cluster_2_distal_link: geometry collision mesh filename=package://meshes/665_meshes/distal_link.STL; visual mesh filename=package://meshes/665_meshes/distal_link.STL
- link cluster_2_end_link: geometry collision mesh filename=package://meshes/665_meshes/end_link.STL; visual mesh filename=package://meshes/665_meshes/end_link.STL
- link cluster_2_proximal_link: geometry collision mesh filename=package://meshes/665_meshes/proximal_link.STL; visual mesh filename=package://meshes/665_meshes/proximal_link.STL
- link cluster_3_distal_link: geometry collision mesh filename=package://meshes/5555_meshes/distal_link.STL; visual mesh filename=package://meshes/5555_meshes/distal_link.STL
- link cluster_3_proximal_link: geometry collision mesh filename=package://meshes/5555_meshes/proximal_link.STL; visual mesh filename=package://meshes/5555_meshes/proximal_link.STL
- link cluster_3_wrist_link: geometry collision mesh filename=package://meshes/5555_meshes/wrist_link.STL; visual mesh filename=package://meshes/5555_meshes/wrist_link.STL
