Commit message: commenting torso stuff back in and updated crab mass properties, still getting errors about parts not having mass properties

File: robot_model/crab/crab_old.urdf (robot description, URDF)
Before this commit: robot crab_robot, 73 links, 72 joints
Links:
- link base_footprint: mass 1e-10 -> None
