Commit message: Create crab interface and update link and joint indices

File: robot_model/crab/crab.urdf (robot description, URDF)
Before this commit: robot crab, 61 links, 60 joints
Links:
- added link back_left_hip_link
- added link back_right_hip_link
- added link front_left_hip_link
- added link front_right_hip_link
- added link imu, mass 0
- link body: geometry collision box size=3 5 0.5; visual box size=3 5 0.5
Joints:
- removed joint back_left_base_fix
- removed joint back_right_base_fix
- removed joint front_left_base_fix
- removed joint front_right_base_fix
- added joint back_left_hip_pitch: type revolute, parent body, child back_left_base_link, origin xyz=-1.5 -2.4 0 rpy=0 3.14 0, axis 1 0 0, limit lower=-1.57 upper=1.57 effort=0 velocity=0
- added joint back_left_hip_yaw: type revolute, parent back_left_base_link, child back_left_hip_link, origin xyz=0 0 0 rpy=0 0 0, axis 0 1 0, limit lower=0 upper=1.57 effort=0 velocity=0
- added joint back_right_hip_pitch: type revolute, parent body, child back_right_base_link, origin xyz=1.5 -2.4 0 rpy=0 3.14 0, axis 1 0 0, limit lower=-1.57 upper=1.57 effort=0 velocity=0
- added joint back_right_hip_yaw: type revolute, parent back_right_base_link, child back_right_hip_link, origin xyz=0 0 0 rpy=0 0 0, axis 0 1 0, limit lower=-1.57 upper=0 effort=0 velocity=0
- added joint front_left_hip_pitch: type revolute, parent body, child front_left_base_link, origin xyz=-1.5 2.4 0 rpy=0 3.14 0, axis 1 0 0, limit lower=-1.57 upper=1.57 effort=0 velocity=0
- added joint front_left_hip_yaw: type revolute, parent front_left_base_link, child front_left_hip_link, origin xyz=0 0 0 rpy=0 0 0, axis 0 1 0, limit lower=0 upper=1.57 effort=0 velocity=0
- added joint front_right_hip_pitch: type revolute, parent body, child front_right_base_link, origin xyz=1.5 2.4 0 rpy=0 3.14 0, axis 1 0 0, limit lower=-1.57 upper=1.57 effort=0 velocity=0
- added joint front_right_hip_yaw: type revolute, parent front_right_base_link, child front_right_hip_link, origin xyz=0 0 0 rpy=0 0 0, axis 0 1 0, limit lower=-1.57 upper=0 effort=0 velocity=0
- added joint imu_joint: type fixed, parent body, child imu, origin xyz=1.5 2.5 0.25 rpy=0 0 0, axis 0 0 0
- joint back_left_cluster_1_base_fix: parent back_left_base_link -> back_left_hip_link
- joint back_right_cluster_1_base_fix: parent back_right_base_link -> back_right_hip_link
- joint front_left_cluster_1_base_fix: parent front_left_base_link -> front_left_hip_link
- joint front_right_cluster_1_base_fix: parent front_right_base_link -> front_right_hip_link

File: robot_model/crab/rad_arm.urdf (robot description, URDF)
Before this commit: robot rad_arm, 15 links, 14 joints
Links:
- link cluster_1_distal_link: geometry collision mesh filename=package://meshes/776_meshes/distal_link.STL; visual mesh filename=package://meshes/776_meshes/distal_link.STL
- link cluster_1_end_link: geometry collision mesh filename=package://meshes/776_meshes/end_link.STL; visual mesh filename=package://meshes/776_meshes/end_link.STL
- link cluster_1_proximal_link: geometry collision mesh filename=package://meshes/776_meshes/proximal_link.STL; visual mesh filename=package://meshes/776_meshes/proximal_link.STL
- link cluster_2_distal_link: geometry collision mesh filename=package://meshes/665_meshes/distal_link.STL; visual mesh filename=package://meshes/665_meshes/distal_link.STL
- link cluster_2_end_link: geometry collision mesh filename=package://meshes/665_meshes/end_link.STL; visual mesh filename=package://meshes/665_meshes/end_link.STL
- link cluster_2_proximal_link: geometry collision mesh filename=package://meshes/665_meshes/proximal_link.STL; visual mesh filename=package://meshes/665_meshes/proximal_link.STL
- link cluster_3_distal_link: geometry collision mesh filename=package://meshes/5555_meshes/distal_link.STL; visual mesh filename=package://meshes/5555_meshes/distal_link.STL
- link cluster_3_proximal_link: geometry collision mesh filename=package://meshes/5555_meshes/proximal_link.STL; visual mesh filename=package://meshes/5555_meshes/proximal_link.STL
- link cluster_3_wrist_link: geometry collision mesh filename=package://meshes/5555_meshes/wrist_link.STL; visual mesh filename=package://meshes/5555_meshes/wrist_link.STL
