Commit message: updated crab.urdf model with colored body and draco_test_cmds.py

File: robot_model/crab/crab.urdf (robot description, URDF)
Before this commit: robot crab, 61 links, 60 joints
Links:
- removed link back_left_base_link
- removed link back_left_cluster_1_base_link
- removed link back_left_cluster_1_distal_link
- removed link back_left_cluster_1_end_link
- removed link back_left_cluster_1_proximal_link
- removed link back_left_cluster_2_base_link
- removed link back_left_cluster_2_distal_link
- removed link back_left_cluster_2_end_link
- removed link back_left_cluster_2_proximal_link
- removed link back_left_cluster_3_base_link
- removed link back_left_cluster_3_distal_link
- removed link back_left_cluster_3_end_link
- removed link back_left_cluster_3_mid_link
- removed link back_left_cluster_3_proximal_link
- removed link back_left_cluster_3_wrist_link
- removed link back_right_base_link
- removed link back_right_cluster_1_base_link
- removed link back_right_cluster_1_distal_link
- removed link back_right_cluster_1_end_link
- removed link back_right_cluster_1_proximal_link
- removed link back_right_cluster_2_base_link
- removed link back_right_cluster_2_distal_link
- removed link back_right_cluster_2_end_link
- removed link back_right_cluster_2_proximal_link
- removed link back_right_cluster_3_base_link
- removed link back_right_cluster_3_distal_link
- removed link back_right_cluster_3_end_link
- removed link back_right_cluster_3_mid_link
- removed link back_right_cluster_3_proximal_link
- removed link back_right_cluster_3_wrist_link
- removed link body
- removed link front_left_base_link
- removed link front_left_cluster_1_base_link
- removed link front_left_cluster_1_distal_link
- removed link front_left_cluster_1_end_link
- removed link front_left_cluster_1_proximal_link
- removed link front_left_cluster_2_base_link
- removed link front_left_cluster_2_distal_link
- removed link front_left_cluster_2_end_link
- removed link front_left_cluster_2_proximal_link
- removed link front_left_cluster_3_base_link
- removed link front_left_cluster_3_distal_link
- removed link front_left_cluster_3_end_link
- removed link front_left_cluster_3_mid_link
- removed link front_left_cluster_3_proximal_link
- removed link front_left_cluster_3_wrist_link
- removed link front_right_base_link
- removed link front_right_cluster_1_base_link
- removed link front_right_cluster_1_distal_link
- removed link front_right_cluster_1_end_link
- removed link front_right_cluster_1_proximal_link
- removed link front_right_cluster_2_base_link
- removed link front_right_cluster_2_distal_link
- removed link front_right_cluster_2_end_link
- removed link front_right_cluster_2_proximal_link
- removed link front_right_cluster_3_base_link
- removed link front_right_cluster_3_distal_link
- removed link front_right_cluster_3_end_link
- removed link front_right_cluster_3_mid_link
- removed link front_right_cluster_3_proximal_link
- removed link front_right_cluster_3_wrist_link
- added link back__sensor_link; visual box size=0.45 0.075 0.1
- added link back_left__base_link
- added link back_left__cluster_1_base_link, mass 3; collision cylinder length=0.5 radius=0.127; visual cylinder length=0.5 radius=0.127
- added link back_left__cluster_1_distal_link, mass 5.08924821549112; collision mesh filename=package://meshes/776_meshes/distal_link.STL; visual mesh filename=package://meshes/776_meshes/distal_link.STL
- added link back_left__cluster_1_end_link, mass 0.581661203844435; collision mesh filename=package://meshes/776_meshes/end_link.STL; visual mesh filename=package://meshes/776_meshes/end_link.STL
- added link back_left__cluster_1_proximal_link, mass 16.527; collision mesh filename=package://meshes/776_meshes/proximal_link.STL; visual mesh filename=package://meshes/776_meshes/proximal_link.STL
- added link back_left__cluster_2_base_link, mass 3; collision cylinder length=0.5 radius=0.1016; visual cylinder length=0.5 radius=0.1016
- added link back_left__cluster_2_distal_link, mass 4.0284; collision mesh filename=package://meshes/665_meshes/distal_link.STL; visual mesh filename=package://meshes/665_meshes/distal_link.STL
- added link back_left__cluster_2_end_link, mass 0.55563; collision mesh filename=package://meshes/665_meshes/end_link.STL; visual mesh filename=package://meshes/665_meshes/end_link.STL
- added link back_left__cluster_2_proximal_link, mass 10.138; collision mesh filename=package://meshes/665_meshes/proximal_link.STL; visual mesh filename=package://meshes/665_meshes/proximal_link.STL
- added link back_left__cluster_3_base_link, mass 3; collision cylinder length=0.5 radius=0.092075; visual cylinder length=0.5 radius=0.092075
- added link back_left__cluster_3_distal_link, mass 3.9917; collision mesh filename=package://meshes/5555_meshes/distal_link.STL; visual mesh filename=package://meshes/5555_meshes/distal_link.STL
- added link back_left__cluster_3_end_link
- added link back_left__cluster_3_mid_link, mass 3; collision cylinder length=0.5 radius=0.092075; visual cylinder length=0.5 radius=0.092075
- added link back_left__cluster_3_proximal_link, mass 9.0522; collision mesh filename=package://meshes/5555_meshes/proximal_link.STL; visual mesh filename=package://meshes/5555_meshes/proximal_link.STL
- added link back_left__cluster_3_wrist_link, mass 2.5013; collision mesh filename=package://meshes/5555_meshes/wrist_link.STL; visual mesh filename=package://meshes/5555_meshes/wrist_link.STL
- added link back_right__base_link
- added link back_right__cluster_1_base_link, mass 3; collision cylinder length=0.5 radius=0.127; visual cylinder length=0.5 radius=0.127
- added link back_right__cluster_1_distal_link, mass 5.08924821549112; collision mesh filename=package://meshes/776_meshes/distal_link.STL; visual mesh filename=package://meshes/776_meshes/distal_link.STL
- added link back_right__cluster_1_end_link, mass 0.581661203844435; collision mesh filename=package://meshes/776_meshes/end_link.STL; visual mesh filename=package://meshes/776_meshes/end_link.STL
- added link back_right__cluster_1_proximal_link, mass 16.527; collision mesh filename=package://meshes/776_meshes/proximal_link.STL; visual mesh filename=package://meshes/776_meshes/proximal_link.STL
- added link back_right__cluster_2_base_link, mass 3; collision cylinder length=0.5 radius=0.1016; visual cylinder length=0.5 radius=0.1016
- added link back_right__cluster_2_distal_link, mass 4.0284; collision mesh filename=package://meshes/665_meshes/distal_link.STL; visual mesh filename=package://meshes/665_meshes/distal_link.STL
- added link back_right__cluster_2_end_link, mass 0.55563; collision mesh filename=package://meshes/665_meshes/end_link.STL; visual mesh filename=package://meshes/665_meshes/end_link.STL
- added link back_right__cluster_2_proximal_link, mass 10.138; collision mesh filename=package://meshes/665_meshes/proximal_link.STL; visual mesh filename=package://meshes/665_meshes/proximal_link.STL
- added link back_right__cluster_3_base_link, mass 3; collision cylinder length=0.5 radius=0.092075; visual cylinder length=0.5 radius=0.092075
- added link back_right__cluster_3_distal_link, mass 3.9917; collision mesh filename=package://meshes/5555_meshes/distal_link.STL; visual mesh filename=package://meshes/5555_meshes/distal_link.STL
- added link back_right__cluster_3_end_link
- added link back_right__cluster_3_mid_link, mass 3; collision cylinder length=0.5 radius=0.092075; visual cylinder length=0.5 radius=0.092075
- added link back_right__cluster_3_proximal_link, mass 9.0522; collision mesh filename=package://meshes/5555_meshes/proximal_link.STL; visual mesh filename=package://meshes/5555_meshes/proximal_link.STL
- added link back_right__cluster_3_wrist_link, mass 2.5013; collision mesh filename=package://meshes/5555_meshes/wrist_link.STL; visual mesh filename=package://meshes/5555_meshes/wrist_link.STL
- added link base_footprint
- added link base_link, mass 1; collision mesh filename=package://meshes/base_link/base_link.stl scale=1 1 1; visual mesh filename=package://meshes/base_link/base_link.stl scale=1 1 1
- added link front_left__base_link
- added link front_left__cluster_1_base_link, mass 3; collision cylinder length=0.5 radius=0.127; visual cylinder length=0.5 radius=0.127
- added link front_left__cluster_1_distal_link, mass 5.08924821549112; collision mesh filename=package://meshes/776_meshes/distal_link.STL; visual mesh filename=package://meshes/776_meshes/distal_link.STL
- added link front_left__cluster_1_end_link, mass 0.581661203844435; collision mesh filename=package://meshes/776_meshes/end_link.STL; visual mesh filename=package://meshes/776_meshes/end_link.STL
- added link front_left__cluster_1_proximal_link, mass 16.527; collision mesh filename=package://meshes/776_meshes/proximal_link.STL; visual mesh filename=package://meshes/776_meshes/proximal_link.STL
- added link front_left__cluster_2_base_link, mass 3; collision cylinder length=0.5 radius=0.1016; visual cylinder length=0.5 radius=0.1016
- added link front_left__cluster_2_distal_link, mass 4.0284; collision mesh filename=package://meshes/665_meshes/distal_link.STL; visual mesh filename=package://meshes/665_meshes/distal_link.STL
- added link front_left__cluster_2_end_link, mass 0.55563; collision mesh filename=package://meshes/665_meshes/end_link.STL; visual mesh filename=package://meshes/665_meshes/end_link.STL
- added link front_left__cluster_2_proximal_link, mass 10.138; collision mesh filename=package://meshes/665_meshes/proximal_link.STL; visual mesh filename=package://meshes/665_meshes/proximal_link.STL
- added link front_left__cluster_3_base_link, mass 3; collision cylinder length=0.5 radius=0.092075; visual cylinder length=0.5 radius=0.092075
- added link front_left__cluster_3_distal_link, mass 3.9917; collision mesh filename=package://meshes/5555_meshes/distal_link.STL; visual mesh filename=package://meshes/5555_meshes/distal_link.STL
- added link front_left__cluster_3_end_link
- added link front_left__cluster_3_mid_link, mass 3; collision cylinder length=0.5 radius=0.092075; visual cylinder length=0.5 radius=0.092075
- added link front_left__cluster_3_proximal_link, mass 9.0522; collision mesh filename=package://meshes/5555_meshes/proximal_link.STL; visual mesh filename=package://meshes/5555_meshes/proximal_link.STL
- added link front_left__cluster_3_wrist_link, mass 2.5013; collision mesh filename=package://meshes/5555_meshes/wrist_link.STL; visual mesh filename=package://meshes/5555_meshes/wrist_link.STL
- added link front_left__sensor_link; visual box size=0.4 0.075 0.1
- added link front_right__base_link
- added link front_right__cluster_1_base_link, mass 3; collision cylinder length=0.5 radius=0.127; visual cylinder length=0.5 radius=0.127
- added link front_right__cluster_1_distal_link, mass 5.08924821549112; collision mesh filename=package://meshes/776_meshes/distal_link.STL; visual mesh filename=package://meshes/776_meshes/distal_link.STL
- added link front_right__cluster_1_end_link, mass 0.581661203844435; collision mesh filename=package://meshes/776_meshes/end_link.STL; visual mesh filename=package://meshes/776_meshes/end_link.STL
- added link front_right__cluster_1_proximal_link, mass 16.527; collision mesh filename=package://meshes/776_meshes/proximal_link.STL; visual mesh filename=package://meshes/776_meshes/proximal_link.STL
- added link front_right__cluster_2_base_link, mass 3; collision cylinder length=0.5 radius=0.1016; visual cylinder length=0.5 radius=0.1016
- added link front_right__cluster_2_distal_link, mass 4.0284; collision mesh filename=package://meshes/665_meshes/distal_link.STL; visual mesh filename=package://meshes/665_meshes/distal_link.STL
- added link front_right__cluster_2_end_link, mass 0.55563; collision mesh filename=package://meshes/665_meshes/end_link.STL; visual mesh filename=package://meshes/665_meshes/end_link.STL
- added link front_right__cluster_2_proximal_link, mass 10.138; collision mesh filename=package://meshes/665_meshes/proximal_link.STL; visual mesh filename=package://meshes/665_meshes/proximal_link.STL
- added link front_right__cluster_3_base_link, mass 3; collision cylinder length=0.5 radius=0.092075; visual cylinder length=0.5 radius=0.092075
- added link front_right__cluster_3_distal_link, mass 3.9917; collision mesh filename=package://meshes/5555_meshes/distal_link.STL; visual mesh filename=package://meshes/5555_meshes/distal_link.STL
- added link front_right__cluster_3_end_link
- added link front_right__cluster_3_mid_link, mass 3; collision cylinder length=0.5 radius=0.092075; visual cylinder length=0.5 radius=0.092075
- added link front_right__cluster_3_proximal_link, mass 9.0522; collision mesh filename=package://meshes/5555_meshes/proximal_link.STL; visual mesh filename=package://meshes/5555_meshes/proximal_link.STL
- added link front_right__cluster_3_wrist_link, mass 2.5013; collision mesh filename=package://meshes/5555_meshes/wrist_link.STL; visual mesh filename=package://meshes/5555_meshes/wrist_link.STL
- added link front_right__sensor_link; visual box size=0.4 0.075 0.1
- added link left__sensor_link; visual box size=0.075 0.45 0.1
- added link lidar_link; visual cylinder length=0.1 radius=0.25
- added link right__sensor_link; visual box size=0.075 0.45 0.1
Joints:
- removed joint back_left_base_fix
- removed joint back_left_cluster_1_base_fix
- removed joint back_left_cluster_1_end_joint
- removed joint back_left_cluster_1_pitch
- removed joint back_left_cluster_1_roll
- removed joint back_left_cluster_2_base_fix
- removed joint back_left_cluster_2_end_joint
- removed joint back_left_cluster_2_pitch
- removed joint back_left_cluster_2_roll
- removed joint back_left_cluster_3_base_fix
- removed joint back_left_cluster_3_end_joint
- removed joint back_left_cluster_3_mid_joint
- removed joint back_left_cluster_3_pitch
- removed joint back_left_cluster_3_roll
- removed joint back_left_cluster_3_wrist
- removed joint back_right_base_fix
- removed joint back_right_cluster_1_base_fix
- removed joint back_right_cluster_1_end_joint
- removed joint back_right_cluster_1_pitch
- removed joint back_right_cluster_1_roll
- removed joint back_right_cluster_2_base_fix
- removed joint back_right_cluster_2_end_joint
- removed joint back_right_cluster_2_pitch
- removed joint back_right_cluster_2_roll
- removed joint back_right_cluster_3_base_fix
- removed joint back_right_cluster_3_end_joint
- removed joint back_right_cluster_3_mid_joint
- removed joint back_right_cluster_3_pitch
- removed joint back_right_cluster_3_roll
- removed joint back_right_cluster_3_wrist
- removed joint front_left_base_fix
- removed joint front_left_cluster_1_base_fix
- removed joint front_left_cluster_1_end_joint
- removed joint front_left_cluster_1_pitch
- removed joint front_left_cluster_1_roll
- removed joint front_left_cluster_2_base_fix
- removed joint front_left_cluster_2_end_joint
- removed joint front_left_cluster_2_pitch
- removed joint front_left_cluster_2_roll
- removed joint front_left_cluster_3_base_fix
- removed joint front_left_cluster_3_end_joint
- removed joint front_left_cluster_3_mid_joint
- removed joint front_left_cluster_3_pitch
- removed joint front_left_cluster_3_roll
- removed joint front_left_cluster_3_wrist
- removed joint front_right_base_fix
- removed joint front_right_cluster_1_base_fix
- removed joint front_right_cluster_1_end_joint
- removed joint front_right_cluster_1_pitch
- removed joint front_right_cluster_1_roll
- removed joint front_right_cluster_2_base_fix
- removed joint front_right_cluster_2_end_joint
- removed joint front_right_cluster_2_pitch
- removed joint front_right_cluster_2_roll
- removed joint front_right_cluster_3_base_fix
- removed joint front_right_cluster_3_end_joint
- removed joint front_right_cluster_3_mid_joint
- removed joint front_right_cluster_3_pitch
- removed joint front_right_cluster_3_roll
- removed joint front_right_cluster_3_wrist
- added joint back_left__cluster_1_base_fix: type fixed, parent back_left__base_link, child back_left__cluster_1_base_link, origin xyz=0 0 0 rpy=0 0 0
- added joint back_left__cluster_1_end_joint: type fixed, parent back_left__cluster_1_distal_link, child back_left__cluster_1_end_link, origin xyz=-0.134923898079026 0.224014512313731 0 rpy=-1.57079632679489 0 0.0350103166030986, axis 0 0 0
- added joint back_left__cluster_1_pitch: type revolute, parent back_left__cluster_1_proximal_link, child back_left__cluster_1_distal_link, origin xyz=0.127 0 0.34925 rpy=1.57079632679489 0.0350103166030992 0, axis 0 0 1, limit lower=-3.14 upper=0 effort=0 velocity=0
- added joint back_left__cluster_1_roll: type revolute, parent back_left__cluster_1_base_link, child back_left__cluster_1_proximal_link, origin xyz=0 0 0.5 rpy=0 0 0, axis 0 0 1, limit lower=-3.14 upper=3.14 effort=0 velocity=0
- added joint back_left__cluster_2_base_fix: type fixed, parent back_left__cluster_1_end_link, child back_left__cluster_2_base_link, origin xyz=0 0 0 rpy=0 0 0
- added joint back_left__cluster_2_end_joint: type fixed, parent back_left__cluster_2_distal_link, child back_left__cluster_2_end_link, origin xyz=-0.1016 0.2032 0 rpy=-1.5708 0 0, axis 0 0 0
- added joint back_left__cluster_2_pitch: type revolute, parent back_left__cluster_2_proximal_link, child back_left__cluster_2_distal_link, origin xyz=0.1016 0 0.34925 rpy=1.5708 0 0, axis 0 0 1, limit lower=-3.14 upper=0 effort=0 velocity=0
- added joint back_left__cluster_2_roll: type revolute, parent back_left__cluster_2_base_link, child back_left__cluster_2_proximal_link, origin xyz=0 0 0.5 rpy=0 0 0, axis 0 0 1, limit lower=-3.14 upper=3.14 effort=0 velocity=0
- added joint back_left__cluster_3_base_fix: type fixed, parent back_left__cluster_2_end_link, child back_left__cluster_3_base_link, origin xyz=0 0 0 rpy=0 0 0
- added joint back_left__cluster_3_end_joint: type fixed, parent back_left__cluster_3_wrist_link, child back_left__cluster_3_end_link, origin xyz=0 0 0.082551 rpy=0 0 0, axis 0 0 0
- added joint back_left__cluster_3_mid_joint: type fixed, parent back_left__cluster_3_distal_link, child back_left__cluster_3_mid_link, origin xyz=-0.0889 0.2032 0 rpy=-1.5708 0 0, axis 0 0 0
- added joint back_left__cluster_3_pitch: type revolute, parent back_left__cluster_3_proximal_link, child back_left__cluster_3_distal_link, origin xyz=0.0889 0 0.34925 rpy=1.5708 0 0, axis 0 0 1, limit lower=-3.14 upper=0 effort=0 velocity=0
- added joint back_left__cluster_3_roll: type revolute, parent back_left__cluster_3_base_link, child back_left__cluster_3_proximal_link, origin xyz=0 0 0.5 rpy=0 0 0, axis 0 0 1, limit lower=-3.14 upper=3.14 effort=0 velocity=0
- added joint back_left__cluster_3_wrist: type revolute, parent back_left__cluster_3_mid_link, child back_left__cluster_3_wrist_link, origin xyz=0 0 0.5 rpy=0 0 0, axis 0 0 1, limit lower=-3.14 upper=3.14 effort=0 velocity=0
- added joint back_right__cluster_1_base_fix: type fixed, parent back_right__base_link, child back_right__cluster_1_base_link, origin xyz=0 0 0 rpy=0 0 0
- added joint back_right__cluster_1_end_joint: type fixed, parent back_right__cluster_1_distal_link, child back_right__cluster_1_end_link, origin xyz=-0.134923898079026 0.224014512313731 0 rpy=-1.57079632679489 0 0.0350103166030986, axis 0 0 0
- added joint back_right__cluster_1_pitch: type revolute, parent back_right__cluster_1_proximal_link, child back_right__cluster_1_distal_link, origin xyz=0.127 0 0.34925 rpy=1.57079632679489 0.0350103166030992 0, axis 0 0 1, limit lower=-3.14 upper=0 effort=0 velocity=0
- added joint back_right__cluster_1_roll: type revolute, parent back_right__cluster_1_base_link, child back_right__cluster_1_proximal_link, origin xyz=0 0 0.5 rpy=0 0 0, axis 0 0 1, limit lower=-3.14 upper=3.14 effort=0 velocity=0
- added joint back_right__cluster_2_base_fix: type fixed, parent back_right__cluster_1_end_link, child back_right__cluster_2_base_link, origin xyz=0 0 0 rpy=0 0 0
- added joint back_right__cluster_2_end_joint: type fixed, parent back_right__cluster_2_distal_link, child back_right__cluster_2_end_link, origin xyz=-0.1016 0.2032 0 rpy=-1.5708 0 0, axis 0 0 0
- added joint back_right__cluster_2_pitch: type revolute, parent back_right__cluster_2_proximal_link, child back_right__cluster_2_distal_link, origin xyz=0.1016 0 0.34925 rpy=1.5708 0 0, axis 0 0 1, limit lower=-3.14 upper=0 effort=0 velocity=0
- added joint back_right__cluster_2_roll: type revolute, parent back_right__cluster_2_base_link, child back_right__cluster_2_proximal_link, origin xyz=0 0 0.5 rpy=0 0 0, axis 0 0 1, limit lower=-3.14 upper=3.14 effort=0 velocity=0
- added joint back_right__cluster_3_base_fix: type fixed, parent back_right__cluster_2_end_link, child back_right__cluster_3_base_link, origin xyz=0 0 0 rpy=0 0 0
- added joint back_right__cluster_3_end_joint: type fixed, parent back_right__cluster_3_wrist_link, child back_right__cluster_3_end_link, origin xyz=0 0 0.082551 rpy=0 0 0, axis 0 0 0
- added joint back_right__cluster_3_mid_joint: type fixed, parent back_right__cluster_3_distal_link, child back_right__cluster_3_mid_link, origin xyz=-0.0889 0.2032 0 rpy=-1.5708 0 0, axis 0 0 0
- added joint back_right__cluster_3_pitch: type revolute, parent back_right__cluster_3_proximal_link, child back_right__cluster_3_distal_link, origin xyz=0.0889 0 0.34925 rpy=1.5708 0 0, axis 0 0 1, limit lower=-3.14 upper=0 effort=0 velocity=0
- added joint back_right__cluster_3_roll: type revolute, parent back_right__cluster_3_base_link, child back_right__cluster_3_proximal_link, origin xyz=0 0 0.5 rpy=0 0 0, axis 0 0 1, limit lower=-3.14 upper=3.14 effort=0 velocity=0
- added joint back_right__cluster_3_wrist: type revolute, parent back_right__cluster_3_mid_link, child back_right__cluster_3_wrist_link, origin xyz=0 0 0.5 rpy=0 0 0, axis 0 0 1, limit lower=-3.14 upper=3.14 effort=0 velocity=0
- added joint base_joint: type fixed, parent base_footprint, child base_link, origin xyz=0 0 0 rpy=0 0 0
- added joint base_link_back__sensor_joint: type fixed, parent base_link, child back__sensor_link, origin xyz=0 -1.5 0 rpy=0 0 0
- added joint base_link_back_left__joint: type fixed, parent base_link, child back_left__base_link, origin xyz=-1.0 -1.0 0 rpy=3.14 1.57 0
- added joint base_link_back_right__joint: type fixed, parent base_link, child back_right__base_link, origin xyz=1.0 -1.0 0 rpy=0 1.57 0
- added joint base_link_front_left__joint: type fixed, parent base_link, child front_left__base_link, origin xyz=-1.0 1.0 0 rpy=3.14 1.57 0
- added joint base_link_front_left__sensor_joint: type fixed, parent base_link, child front_left__sensor_link, origin xyz=-0.725 1.5 0 rpy=0 0 0
- added joint base_link_front_right__joint: type fixed, parent base_link, child front_right__base_link, origin xyz=1.0 1.0 0 rpy=0 1.57 0
- added joint base_link_front_right__sensor_joint: type fixed, parent base_link, child front_right__sensor_link, origin xyz=0.725 1.5 0 rpy=0 0 0
- added joint base_link_left__sensor_joint: type fixed, parent base_link, child left__sensor_link, origin xyz=-1.0 0 0 rpy=0 0 0
- added joint base_link_right__sensor_joint: type fixed, parent base_link, child right__sensor_link, origin xyz=1.0 0 0 rpy=0 0 0
- added joint front_left__cluster_1_base_fix: type fixed, parent front_left__base_link, child front_left__cluster_1_base_link, origin xyz=0 0 0 rpy=0 0 0
- added joint front_left__cluster_1_end_joint: type fixed, parent front_left__cluster_1_distal_link, child front_left__cluster_1_end_link, origin xyz=-0.134923898079026 0.224014512313731 0 rpy=-1.57079632679489 0 0.0350103166030986, axis 0 0 0
- added joint front_left__cluster_1_pitch: type revolute, parent front_left__cluster_1_proximal_link, child front_left__cluster_1_distal_link, origin xyz=0.127 0 0.34925 rpy=1.57079632679489 0.0350103166030992 0, axis 0 0 1, limit lower=-3.14 upper=0 effort=0 velocity=0
- added joint front_left__cluster_1_roll: type revolute, parent front_left__cluster_1_base_link, child front_left__cluster_1_proximal_link, origin xyz=0 0 0.5 rpy=0 0 0, axis 0 0 1, limit lower=-3.14 upper=3.14 effort=0 velocity=0
- added joint front_left__cluster_2_base_fix: type fixed, parent front_left__cluster_1_end_link, child front_left__cluster_2_base_link, origin xyz=0 0 0 rpy=0 0 0
- added joint front_left__cluster_2_end_joint: type fixed, parent front_left__cluster_2_distal_link, child front_left__cluster_2_end_link, origin xyz=-0.1016 0.2032 0 rpy=-1.5708 0 0, axis 0 0 0
- added joint front_left__cluster_2_pitch: type revolute, parent front_left__cluster_2_proximal_link, child front_left__cluster_2_distal_link, origin xyz=0.1016 0 0.34925 rpy=1.5708 0 0, axis 0 0 1, limit lower=-3.14 upper=0 effort=0 velocity=0
- added joint front_left__cluster_2_roll: type revolute, parent front_left__cluster_2_base_link, child front_left__cluster_2_proximal_link, origin xyz=0 0 0.5 rpy=0 0 0, axis 0 0 1, limit lower=-3.14 upper=3.14 effort=0 velocity=0
- added joint front_left__cluster_3_base_fix: type fixed, parent front_left__cluster_2_end_link, child front_left__cluster_3_base_link, origin xyz=0 0 0 rpy=0 0 0
- added joint front_left__cluster_3_end_joint: type fixed, parent front_left__cluster_3_wrist_link, child front_left__cluster_3_end_link, origin xyz=0 0 0.082551 rpy=0 0 0, axis 0 0 0
- added joint front_left__cluster_3_mid_joint: type fixed, parent front_left__cluster_3_distal_link, child front_left__cluster_3_mid_link, origin xyz=-0.0889 0.2032 0 rpy=-1.5708 0 0, axis 0 0 0
- added joint front_left__cluster_3_pitch: type revolute, parent front_left__cluster_3_proximal_link, child front_left__cluster_3_distal_link, origin xyz=0.0889 0 0.34925 rpy=1.5708 0 0, axis 0 0 1, limit lower=-3.14 upper=0 effort=0 velocity=0
- added joint front_left__cluster_3_roll: type revolute, parent front_left__cluster_3_base_link, child front_left__cluster_3_proximal_link, origin xyz=0 0 0.5 rpy=0 0 0, axis 0 0 1, limit lower=-3.14 upper=3.14 effort=0 velocity=0
- added joint front_left__cluster_3_wrist: type revolute, parent front_left__cluster_3_mid_link, child front_left__cluster_3_wrist_link, origin xyz=0 0 0.5 rpy=0 0 0, axis 0 0 1, limit lower=-3.14 upper=3.14 effort=0 velocity=0
- added joint front_right__cluster_1_base_fix: type fixed, parent front_right__base_link, child front_right__cluster_1_base_link, origin xyz=0 0 0 rpy=0 0 0
- added joint front_right__cluster_1_end_joint: type fixed, parent front_right__cluster_1_distal_link, child front_right__cluster_1_end_link, origin xyz=-0.134923898079026 0.224014512313731 0 rpy=-1.57079632679489 0 0.0350103166030986, axis 0 0 0
- added joint front_right__cluster_1_pitch: type revolute, parent front_right__cluster_1_proximal_link, child front_right__cluster_1_distal_link, origin xyz=0.127 0 0.34925 rpy=1.57079632679489 0.0350103166030992 0, axis 0 0 1, limit lower=-3.14 upper=0 effort=0 velocity=0
- added joint front_right__cluster_1_roll: type revolute, parent front_right__cluster_1_base_link, child front_right__cluster_1_proximal_link, origin xyz=0 0 0.5 rpy=0 0 0, axis 0 0 1, limit lower=-3.14 upper=3.14 effort=0 velocity=0
- added joint front_right__cluster_2_base_fix: type fixed, parent front_right__cluster_1_end_link, child front_right__cluster_2_base_link, origin xyz=0 0 0 rpy=0 0 0
- added joint front_right__cluster_2_end_joint: type fixed, parent front_right__cluster_2_distal_link, child front_right__cluster_2_end_link, origin xyz=-0.1016 0.2032 0 rpy=-1.5708 0 0, axis 0 0 0
- added joint front_right__cluster_2_pitch: type revolute, parent front_right__cluster_2_proximal_link, child front_right__cluster_2_distal_link, origin xyz=0.1016 0 0.34925 rpy=1.5708 0 0, axis 0 0 1, limit lower=-3.14 upper=0 effort=0 velocity=0
- added joint front_right__cluster_2_roll: type revolute, parent front_right__cluster_2_base_link, child front_right__cluster_2_proximal_link, origin xyz=0 0 0.5 rpy=0 0 0, axis 0 0 1, limit lower=-3.14 upper=3.14 effort=0 velocity=0
- added joint front_right__cluster_3_base_fix: type fixed, parent front_right__cluster_2_end_link, child front_right__cluster_3_base_link, origin xyz=0 0 0 rpy=0 0 0
- added joint front_right__cluster_3_end_joint: type fixed, parent front_right__cluster_3_wrist_link, child front_right__cluster_3_end_link, origin xyz=0 0 0.082551 rpy=0 0 0, axis 0 0 0
- added joint front_right__cluster_3_mid_joint: type fixed, parent front_right__cluster_3_distal_link, child front_right__cluster_3_mid_link, origin xyz=-0.0889 0.2032 0 rpy=-1.5708 0 0, axis 0 0 0
- added joint front_right__cluster_3_pitch: type revolute, parent front_right__cluster_3_proximal_link, child front_right__cluster_3_distal_link, origin xyz=0.0889 0 0.34925 rpy=1.5708 0 0, axis 0 0 1, limit lower=-3.14 upper=0 effort=0 velocity=0
- added joint front_right__cluster_3_roll: type revolute, parent front_right__cluster_3_base_link, child front_right__cluster_3_proximal_link, origin xyz=0 0 0.5 rpy=0 0 0, axis 0 0 1, limit lower=-3.14 upper=3.14 effort=0 velocity=0
- added joint front_right__cluster_3_wrist: type revolute, parent front_right__cluster_3_mid_link, child front_right__cluster_3_wrist_link, origin xyz=0 0 0.5 rpy=0 0 0, axis 0 0 1, limit lower=-3.14 upper=3.14 effort=0 velocity=0
- added joint lidar_base_joint: type fixed, parent base_link, child lidar_link, origin xyz=0 0 0.25 rpy=0 0 0
