Commit message: updated crab.urdf with magnetic feet end effectors

File: robot_model/crab/crab.urdf (robot description, URDF)
Before this commit: robot crab_robot, 68 links, 67 joints
Links:
- removed link lidar_link
- added link back_left__foot_link; collision box size=0.5 0.5 0.1; visual box size=0.5 0.5 0.1
- added link back_right__foot_link; collision box size=0.5 0.5 0.1; visual box size=0.5 0.5 0.1
- added link bottom_lidar_link; visual cylinder length=0.1 radius=0.25
- added link front_left__foot_link; collision box size=0.5 0.5 0.1; visual box size=0.5 0.5 0.1
- added link front_right__foot_link; collision box size=0.5 0.5 0.1; visual box size=0.5 0.5 0.1
- added link top_lidar_link; visual cylinder length=0.1 radius=0.25
Joints:
- removed joint lidar_base_joint
- added joint back_left__cluster_3_wrist_link_foot_joint: type fixed, parent back_left__cluster_3_wrist_link, child back_left__foot_link, origin xyz=0 0 0.15 rpy=0 0 0
- added joint back_right__cluster_3_wrist_link_foot_joint: type fixed, parent back_right__cluster_3_wrist_link, child back_right__foot_link, origin xyz=0 0 0.15 rpy=0 0 0
- added joint bottom_lidar_base_joint: type fixed, parent base_link, child bottom_lidar_link, origin xyz=0 0 -0.3 rpy=0 0 0
- added joint front_left__cluster_3_wrist_link_foot_joint: type fixed, parent front_left__cluster_3_wrist_link, child front_left__foot_link, origin xyz=0 0 0.15 rpy=0 0 0
- added joint front_right__cluster_3_wrist_link_foot_joint: type fixed, parent front_right__cluster_3_wrist_link, child front_right__foot_link, origin xyz=0 0 0.15 rpy=0 0 0
- added joint top_lidar_base_joint: type fixed, parent base_link, child top_lidar_link, origin xyz=0 0 0.3 rpy=0 0 0

Commit message: fixed land task to rotate feet in direction of landing
also removed hierarchy managers, tuned ihwbc, and added torque and vel
limits to crab.urdf

File: robot_model/crab/crab.urdf (robot description, URDF)
Before this commit: robot crab_robot, 73 links, 72 joints
Joints:
- joint back_left__cluster_1_pitch: limit lower=-3.14 upper=0 effort=0 velocity=0 -> lower=-3.14 upper=0 effort=30 velocity=30
- joint back_left__cluster_1_roll: limit lower=-3.14 upper=3.14 effort=0 velocity=0 -> lower=-3.14 upper=3.14 effort=30 velocity=30
- joint back_left__cluster_2_pitch: limit lower=-3.14 upper=0 effort=0 velocity=0 -> lower=-3.14 upper=0 effort=30 velocity=30
- joint back_left__cluster_2_roll: limit lower=-3.14 upper=3.14 effort=0 velocity=0 -> lower=-3.14 upper=3.14 effort=30 velocity=30
- joint back_left__cluster_3_pitch: limit lower=-3.14 upper=0 effort=0 velocity=0 -> lower=-3.14 upper=0 effort=30 velocity=30
- joint back_left__cluster_3_roll: limit lower=-3.14 upper=3.14 effort=0 velocity=0 -> lower=-3.14 upper=3.14 effort=30 velocity=30
- joint back_left__cluster_3_wrist: limit lower=-3.14 upper=3.14 effort=0 velocity=0 -> lower=-3.14 upper=3.14 effort=30 velocity=30
- joint back_right__cluster_1_pitch: limit lower=-3.14 upper=0 effort=0 velocity=0 -> lower=-3.14 upper=0 effort=30 velocity=30
- joint back_right__cluster_1_roll: limit lower=-3.14 upper=3.14 effort=0 velocity=0 -> lower=-3.14 upper=3.14 effort=30 velocity=30
- joint back_right__cluster_2_pitch: limit lower=-3.14 upper=0 effort=0 velocity=0 -> lower=-3.14 upper=0 effort=30 velocity=30
- joint back_right__cluster_2_roll: limit lower=-3.14 upper=3.14 effort=0 velocity=0 -> lower=-3.14 upper=3.14 effort=30 velocity=30
- joint back_right__cluster_3_pitch: limit lower=-3.14 upper=0 effort=0 velocity=0 -> lower=-3.14 upper=0 effort=30 velocity=30
- joint back_right__cluster_3_roll: limit lower=-3.14 upper=3.14 effort=0 velocity=0 -> lower=-3.14 upper=3.14 effort=30 velocity=30
- joint back_right__cluster_3_wrist: limit lower=-3.14 upper=3.14 effort=0 velocity=0 -> lower=-3.14 upper=3.14 effort=30 velocity=30
- joint front_left__cluster_1_pitch: limit lower=-3.14 upper=0 effort=0 velocity=0 -> lower=-3.14 upper=0 effort=30 velocity=30
- joint front_left__cluster_1_roll: limit lower=-3.14 upper=3.14 effort=0 velocity=0 -> lower=-3.14 upper=3.14 effort=30 velocity=30
- joint front_left__cluster_2_pitch: limit lower=-3.14 upper=0 effort=0 velocity=0 -> lower=-3.14 upper=0 effort=30 velocity=30
- joint front_left__cluster_2_roll: limit lower=-3.14 upper=3.14 effort=0 velocity=0 -> lower=-3.14 upper=3.14 effort=30 velocity=30
- joint front_left__cluster_3_pitch: limit lower=-3.14 upper=0 effort=0 velocity=0 -> lower=-3.14 upper=0 effort=30 velocity=30
- joint front_left__cluster_3_roll: limit lower=-3.14 upper=3.14 effort=0 velocity=0 -> lower=-3.14 upper=3.14 effort=30 velocity=30
- joint front_left__cluster_3_wrist: limit lower=-3.14 upper=3.14 effort=0 velocity=0 -> lower=-3.14 upper=3.14 effort=30 velocity=30
- joint front_right__cluster_1_pitch: limit lower=-3.14 upper=0 effort=0 velocity=0 -> lower=-3.14 upper=0 effort=30 velocity=30
- joint front_right__cluster_1_roll: limit lower=-3.14 upper=3.14 effort=0 velocity=0 -> lower=-3.14 upper=3.14 effort=30 velocity=30
- joint front_right__cluster_2_pitch: limit lower=-3.14 upper=0 effort=0 velocity=0 -> lower=-3.14 upper=0 effort=30 velocity=30
- joint front_right__cluster_2_roll: limit lower=-3.14 upper=3.14 effort=0 velocity=0 -> lower=-3.14 upper=3.14 effort=30 velocity=30
- joint front_right__cluster_3_pitch: limit lower=-3.14 upper=0 effort=0 velocity=0 -> lower=-3.14 upper=0 effort=30 velocity=30
- joint front_right__cluster_3_roll: limit lower=-3.14 upper=3.14 effort=0 velocity=0 -> lower=-3.14 upper=3.14 effort=30 velocity=30
- joint front_right__cluster_3_wrist: limit lower=-3.14 upper=3.14 effort=0 velocity=0 -> lower=-3.14 upper=3.14 effort=30 velocity=30

Commit message: updated with latest crab urdf

File: robot_model/crab/crab.urdf (robot description, URDF)
Before this commit: robot crab_robot, 73 links, 72 joints
Links:
- link back__sensor_link: mass None -> 1
- link base_link: mass 1 -> 100
- link bottom_lidar_link: mass None -> 1
- link front_left__sensor_link: mass None -> 1
- link front_right__sensor_link: mass None -> 1
- link left__sensor_link: mass None -> 1
- link right__sensor_link: mass None -> 1
- link top_lidar_link: mass None -> 1
Joints:
- joint back_left__cluster_1_pitch: limit lower=-3.14 upper=0 effort=30 velocity=30 -> lower=-3.14 upper=0 effort=0 velocity=0
- joint back_left__cluster_1_roll: limit lower=-3.14 upper=3.14 effort=30 velocity=30 -> lower=-3.14 upper=3.14 effort=0 velocity=0
- joint back_left__cluster_2_pitch: limit lower=-3.14 upper=0 effort=30 velocity=30 -> lower=-3.14 upper=0 effort=0 velocity=0
- joint back_left__cluster_2_roll: limit lower=-3.14 upper=3.14 effort=30 velocity=30 -> lower=-3.14 upper=3.14 effort=0 velocity=0
- joint back_left__cluster_3_pitch: limit lower=-3.14 upper=0 effort=30 velocity=30 -> lower=-3.14 upper=0 effort=0 velocity=0
- joint back_left__cluster_3_roll: limit lower=-3.14 upper=3.14 effort=30 velocity=30 -> lower=-3.14 upper=3.14 effort=0 velocity=0
- joint back_left__cluster_3_wrist: limit lower=-3.14 upper=3.14 effort=30 velocity=30 -> lower=-3.14 upper=3.14 effort=0 velocity=0
- joint back_right__cluster_1_pitch: limit lower=-3.14 upper=0 effort=30 velocity=30 -> lower=-3.14 upper=0 effort=0 velocity=0
- joint back_right__cluster_1_roll: limit lower=-3.14 upper=3.14 effort=30 velocity=30 -> lower=-3.14 upper=3.14 effort=0 velocity=0
- joint back_right__cluster_2_pitch: limit lower=-3.14 upper=0 effort=30 velocity=30 -> lower=-3.14 upper=0 effort=0 velocity=0
- joint back_right__cluster_2_roll: limit lower=-3.14 upper=3.14 effort=30 velocity=30 -> lower=-3.14 upper=3.14 effort=0 velocity=0
- joint back_right__cluster_3_pitch: limit lower=-3.14 upper=0 effort=30 velocity=30 -> lower=-3.14 upper=0 effort=0 velocity=0
- joint back_right__cluster_3_roll: limit lower=-3.14 upper=3.14 effort=30 velocity=30 -> lower=-3.14 upper=3.14 effort=0 velocity=0
- joint back_right__cluster_3_wrist: limit lower=-3.14 upper=3.14 effort=30 velocity=30 -> lower=-3.14 upper=3.14 effort=0 velocity=0
- joint front_left__cluster_1_pitch: limit lower=-3.14 upper=0 effort=30 velocity=30 -> lower=-3.14 upper=0 effort=0 velocity=0
- joint front_left__cluster_1_roll: limit lower=-3.14 upper=3.14 effort=30 velocity=30 -> lower=-3.14 upper=3.14 effort=0 velocity=0
- joint front_left__cluster_2_pitch: limit lower=-3.14 upper=0 effort=30 velocity=30 -> lower=-3.14 upper=0 effort=0 velocity=0
- joint front_left__cluster_2_roll: limit lower=-3.14 upper=3.14 effort=30 velocity=30 -> lower=-3.14 upper=3.14 effort=0 velocity=0
- joint front_left__cluster_3_pitch: limit lower=-3.14 upper=0 effort=30 velocity=30 -> lower=-3.14 upper=0 effort=0 velocity=0
- joint front_left__cluster_3_roll: limit lower=-3.14 upper=3.14 effort=30 velocity=30 -> lower=-3.14 upper=3.14 effort=0 velocity=0
- joint front_left__cluster_3_wrist: limit lower=-3.14 upper=3.14 effort=30 velocity=30 -> lower=-3.14 upper=3.14 effort=0 velocity=0
- joint front_right__cluster_1_pitch: limit lower=-3.14 upper=0 effort=30 velocity=30 -> lower=-3.14 upper=0 effort=0 velocity=0
- joint front_right__cluster_1_roll: limit lower=-3.14 upper=3.14 effort=30 velocity=30 -> lower=-3.14 upper=3.14 effort=0 velocity=0
- joint front_right__cluster_2_pitch: limit lower=-3.14 upper=0 effort=30 velocity=30 -> lower=-3.14 upper=0 effort=0 velocity=0
- joint front_right__cluster_2_roll: limit lower=-3.14 upper=3.14 effort=30 velocity=30 -> lower=-3.14 upper=3.14 effort=0 velocity=0
- joint front_right__cluster_3_pitch: limit lower=-3.14 upper=0 effort=30 velocity=30 -> lower=-3.14 upper=0 effort=0 velocity=0
- joint front_right__cluster_3_roll: limit lower=-3.14 upper=3.14 effort=30 velocity=30 -> lower=-3.14 upper=3.14 effort=0 velocity=0
- joint front_right__cluster_3_wrist: limit lower=-3.14 upper=3.14 effort=30 velocity=30 -> lower=-3.14 upper=3.14 effort=0 velocity=0

Commit message: no more errors for back_left & back_right base_link & cluster_3_end_link

File: robot_model/crab/crab.urdf (robot description, URDF)
Before this commit: robot crab_robot, 73 links, 72 joints
Links:
- link back_left__base_link: mass None -> 1e-10
- link back_left__cluster_3_end_link: mass None -> 1e-10
- link back_right__base_link: mass None -> 1e-10
- link back_right__cluster_3_end_link: mass None -> 1e-10

Commit message: added foot link inertias, no more b3Printf errors, but still getting segmentation fault (core dumped) error

File: robot_model/crab/crab.urdf (robot description, URDF)
Before this commit: robot crab_robot, 73 links, 72 joints
Links:
- link back_left__foot_link: mass None -> 1e-10
- link back_right__foot_link: mass None -> 1e-10
- link front_left__foot_link: mass None -> 1e-10
- link front_right__foot_link: mass None -> 1e-10

Commit message: Semi-working rl

File: robot_model/crab/crab.urdf (robot description, URDF)
Before this commit: robot crab_robot, 73 links, 72 joints
Joints:
- joint base_joint: type fixed -> floating

Commit message: Update crab urdf with better meshes

File: robot_model/crab/crab.urdf (robot description, URDF)
Before this commit: robot crab_robot, 73 links, 72 joints
Links:
- link back_left__cluster_1_distal_link: geometry collision mesh filename=package://meshes/cluster_776_distal_link.stl; visual mesh filename=package://meshes/cluster_776_distal_link.stl
- link back_left__cluster_1_end_link: geometry collision mesh filename=package://meshes/cluster_776_end_link.stl; visual mesh filename=package://meshes/cluster_776_end_link.stl
- link back_left__cluster_1_proximal_link: geometry collision mesh filename=package://meshes/cluster_776_proximal_link.stl; visual mesh filename=package://meshes/cluster_776_proximal_link.stl
- link back_left__cluster_2_distal_link: geometry collision mesh filename=package://meshes/cluster_665_distal_link.stl; visual mesh filename=package://meshes/cluster_665_distal_link.stl
- link back_left__cluster_2_end_link: geometry collision mesh filename=package://meshes/cluster_665_end_link.stl; visual mesh filename=package://meshes/cluster_665_end_link.stl
- link back_left__cluster_2_proximal_link: geometry collision mesh filename=package://meshes/cluster_665_proximal_link.stl; visual mesh filename=package://meshes/cluster_665_proximal_link.stl
- link back_left__cluster_3_distal_link: geometry collision mesh filename=package://meshes/cluster_5555_distal_link.stl; visual mesh filename=package://meshes/cluster_5555_distal_link.stl
- link back_left__cluster_3_proximal_link: geometry collision mesh filename=package://meshes/cluster_5555_proximal_link.stl; visual mesh filename=package://meshes/cluster_5555_proximal_link.stl
- link back_left__cluster_3_wrist_link: geometry collision mesh filename=package://meshes/cluster_5555_wrist_link.stl; visual mesh filename=package://meshes/cluster_5555_wrist_link.stl
- link back_left__foot_link: mass 1e-10 -> None
- link back_right__cluster_1_distal_link: geometry collision mesh filename=package://meshes/cluster_776_distal_link.stl; visual mesh filename=package://meshes/cluster_776_distal_link.stl
- link back_right__cluster_1_end_link: geometry collision mesh filename=package://meshes/cluster_776_end_link.stl; visual mesh filename=package://meshes/cluster_776_end_link.stl
- link back_right__cluster_1_proximal_link: geometry collision mesh filename=package://meshes/cluster_776_proximal_link.stl; visual mesh filename=package://meshes/cluster_776_proximal_link.stl
- link back_right__cluster_2_distal_link: geometry collision mesh filename=package://meshes/cluster_665_distal_link.stl; visual mesh filename=package://meshes/cluster_665_distal_link.stl
- link back_right__cluster_2_end_link: geometry collision mesh filename=package://meshes/cluster_665_end_link.stl; visual mesh filename=package://meshes/cluster_665_end_link.stl
- link back_right__cluster_2_proximal_link: geometry collision mesh filename=package://meshes/cluster_665_proximal_link.stl; visual mesh filename=package://meshes/cluster_665_proximal_link.stl
- link back_right__cluster_3_distal_link: geometry collision mesh filename=package://meshes/cluster_5555_distal_link.stl; visual mesh filename=package://meshes/cluster_5555_distal_link.stl
- link back_right__cluster_3_proximal_link: geometry collision mesh filename=package://meshes/cluster_5555_proximal_link.stl; visual mesh filename=package://meshes/cluster_5555_proximal_link.stl
- link back_right__cluster_3_wrist_link: geometry collision mesh filename=package://meshes/cluster_5555_wrist_link.stl; visual mesh filename=package://meshes/cluster_5555_wrist_link.stl
- link back_right__foot_link: mass 1e-10 -> None
- link base_link: geometry collision mesh filename=package://meshes/base_link.stl scale=1 1 1; visual mesh filename=package://meshes/base_link.stl scale=1 1 1
- link front_left__cluster_1_distal_link: geometry collision mesh filename=package://meshes/cluster_776_distal_link.stl; visual mesh filename=package://meshes/cluster_776_distal_link.stl
- link front_left__cluster_1_end_link: geometry collision mesh filename=package://meshes/cluster_776_end_link.stl; visual mesh filename=package://meshes/cluster_776_end_link.stl
- link front_left__cluster_1_proximal_link: geometry collision mesh filename=package://meshes/cluster_776_proximal_link.stl; visual mesh filename=package://meshes/cluster_776_proximal_link.stl
- link front_left__cluster_2_distal_link: geometry collision mesh filename=package://meshes/cluster_665_distal_link.stl; visual mesh filename=package://meshes/cluster_665_distal_link.stl
- link front_left__cluster_2_end_link: geometry collision mesh filename=package://meshes/cluster_665_end_link.stl; visual mesh filename=package://meshes/cluster_665_end_link.stl
- link front_left__cluster_2_proximal_link: geometry collision mesh filename=package://meshes/cluster_665_proximal_link.stl; visual mesh filename=package://meshes/cluster_665_proximal_link.stl
- link front_left__cluster_3_distal_link: geometry collision mesh filename=package://meshes/cluster_5555_distal_link.stl; visual mesh filename=package://meshes/cluster_5555_distal_link.stl
- link front_left__cluster_3_proximal_link: geometry collision mesh filename=package://meshes/cluster_5555_proximal_link.stl; visual mesh filename=package://meshes/cluster_5555_proximal_link.stl
- link front_left__cluster_3_wrist_link: geometry collision mesh filename=package://meshes/cluster_5555_wrist_link.stl; visual mesh filename=package://meshes/cluster_5555_wrist_link.stl
- link front_left__foot_link: mass 1e-10 -> None
- link front_right__cluster_1_distal_link: geometry collision mesh filename=package://meshes/cluster_776_distal_link.stl; visual mesh filename=package://meshes/cluster_776_distal_link.stl
- link front_right__cluster_1_end_link: geometry collision mesh filename=package://meshes/cluster_776_end_link.stl; visual mesh filename=package://meshes/cluster_776_end_link.stl
- link front_right__cluster_1_proximal_link: geometry collision mesh filename=package://meshes/cluster_776_proximal_link.stl; visual mesh filename=package://meshes/cluster_776_proximal_link.stl
- link front_right__cluster_2_distal_link: geometry collision mesh filename=package://meshes/cluster_665_distal_link.stl; visual mesh filename=package://meshes/cluster_665_distal_link.stl
- link front_right__cluster_2_end_link: geometry collision mesh filename=package://meshes/cluster_665_end_link.stl; visual mesh filename=package://meshes/cluster_665_end_link.stl
- link front_right__cluster_2_proximal_link: geometry collision mesh filename=package://meshes/cluster_665_proximal_link.stl; visual mesh filename=package://meshes/cluster_665_proximal_link.stl
- link front_right__cluster_3_distal_link: geometry collision mesh filename=package://meshes/cluster_5555_distal_link.stl; visual mesh filename=package://meshes/cluster_5555_distal_link.stl
- link front_right__cluster_3_proximal_link: geometry collision mesh filename=package://meshes/cluster_5555_proximal_link.stl; visual mesh filename=package://meshes/cluster_5555_proximal_link.stl
- link front_right__cluster_3_wrist_link: geometry collision mesh filename=package://meshes/cluster_5555_wrist_link.stl; visual mesh filename=package://meshes/cluster_5555_wrist_link.stl
- link front_right__foot_link: mass 1e-10 -> None
Joints:
- joint base_joint: type floating -> fixed
