Commit message: modified cylinder.urdf so that it 's bigger

File: robot_model/cylinder.urdf (robot description, URDF)
Before this commit: robot cylinder, 1 links, 0 joints
Links:
- removed link torso_link
- added link cylinder, mass 6.456; collision cylinder length=10 radius=2.0; visual cylinder length=10 radius=2.0
